Commit message: attempt 1

File: models/curiosity_path/urdf/chassis.xacro (robot description, xacro)
@@ -19,5 +19,7 @@
 					rpy="0 0 0"/>
 			<geometry>
-				<mesh filename="package://simulation/models/curiosity_path/meshes/chassis_full_fixed_glitch_v2.dae" scale="${scale_XYZ} ${scale_XYZ} ${scale_XYZ}"/>
+				<!-- This throws an error with O3DE URDF import -->
+				<!-- <mesh filename="package://simulation/models/curiosity_path/meshes/chassis_full_fixed_glitch_v2.dae" scale="${scale_XYZ} ${scale_XYZ} ${scale_XYZ}"/> -->
+				<mesh filename="package://simulation/models/curiosity_path/meshes/chassis_full_fixed_v2.dae" scale="${scale_XYZ} ${scale_XYZ} ${scale_XYZ}"/>
 			</geometry>
 		</collision>
@@ -26,5 +28,6 @@
 					rpy="0 0 0"/>
 			<geometry>
-				<mesh filename="package://simulation/models/curiosity_path/meshes/chassis_full_fixed_glitch_v2.dae" scale="${scale_XYZ} ${scale_XYZ} ${scale_XYZ}"/>
+				<mesh filename="package://simulation/models/curiosity_path/meshes/chassis_full_fixed_v2.dae" scale="${scale_XYZ} ${scale_XYZ} ${scale_XYZ}"/>
+				<!-- <mesh filename="package://simulation/models/curiosity_path/meshes/chassis_full_fixed_glitch_v2.dae" scale="${scale_XYZ} ${scale_XYZ} ${scale_XYZ}"/> -->
 			</geometry>
 		</visual>

Commit message: removed cover_03 from chassis.dae file

File: models/curiosity_path/urdf/chassis.xacro (robot description, xacro)
@@ -19,7 +19,5 @@
 					rpy="0 0 0"/>
 			<geometry>
-				<!-- This throws an error with O3DE URDF import -->
-				<!-- <mesh filename="package://simulation/models/curiosity_path/meshes/chassis_full_fixed_glitch_v2.dae" scale="${scale_XYZ} ${scale_XYZ} ${scale_XYZ}"/> -->
-				<mesh filename="package://simulation/models/curiosity_path/meshes/chassis_full_fixed_v2.dae" scale="${scale_XYZ} ${scale_XYZ} ${scale_XYZ}"/>
+				<mesh filename="package://simulation/models/curiosity_path/meshes/chassis_full_fixed_glitch_v4.dae" scale="${scale_XYZ} ${scale_XYZ} ${scale_XYZ}"/>
 			</geometry>
 		</collision>
@@ -28,6 +26,5 @@
 					rpy="0 0 0"/>
 			<geometry>
-				<mesh filename="package://simulation/models/curiosity_path/meshes/chassis_full_fixed_v2.dae" scale="${scale_XYZ} ${scale_XYZ} ${scale_XYZ}"/>
-				<!-- <mesh filename="package://simulation/models/curiosity_path/meshes/chassis_full_fixed_glitch_v2.dae" scale="${scale_XYZ} ${scale_XYZ} ${scale_XYZ}"/> -->
+				<mesh filename="package://simulation/models/curiosity_path/meshes/chassis_full_fixed_glitch_v4.dae" scale="${scale_XYZ} ${scale_XYZ} ${scale_XYZ}"/>
 			</geometry>
 		</visual>

Commit message: removed cover_03, fixed chassis import

File: models/curiosity_path/urdf/chassis.xacro (robot description, xacro)
@@ -19,5 +19,5 @@
 					rpy="0 0 0"/>
 			<geometry>
-				<mesh filename="package://simulation/models/curiosity_path/meshes/chassis_full_fixed_glitch_v4.dae" scale="${scale_XYZ} ${scale_XYZ} ${scale_XYZ}"/>
+				<mesh filename="package://simulation/models/curiosity_path/meshes/chassis_full_fixed_glitch_v3.dae" scale="${scale_XYZ} ${scale_XYZ} ${scale_XYZ}"/>
 			</geometry>
 		</collision>
@@ -26,5 +26,5 @@
 					rpy="0 0 0"/>
 			<geometry>
-				<mesh filename="package://simulation/models/curiosity_path/meshes/chassis_full_fixed_glitch_v4.dae" scale="${scale_XYZ} ${scale_XYZ} ${scale_XYZ}"/>
+				<mesh filename="package://simulation/models/curiosity_path/meshes/chassis_full_fixed_glitch_v3.dae" scale="${scale_XYZ} ${scale_XYZ} ${scale_XYZ}"/>
 			</geometry>
 		</visual>
